File: m6502-prototyping-board.brd (EAGLE design)
At the start: 110 x 72 mm, 33 parts

Commit message: removed RDY connection to eeprom
Parts:
- removed ROM-RDY: (no value), pinhead:1X02
Connections:
- removed net N$8: EEPROM.1, ROM-RDY.2
- net RDY: no longer ROM-RDY.1
Routing:
- net N$8: track 101.0 -> 0.00 mm, vias 1 -> 0
Changed lines of the file:
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@@
 <element name="U$1" library="holes" library_urn="urn:adsk.eagle:library:237" package="3,2" package3d_urn="urn:adsk.eagle:package:14275/1" value="" x="5.08" y="67.31" smashed="yes"/>
 <element name="U$2" library="holes" library_urn="urn:adsk.eagle:library:237" package="3,2" package3d_urn="urn:adsk.eagle:package:14275/1" value="" x="105.41" y="67.31" smashed="yes"/>
-<element name="ROM-RDY" library="pinhead" library_urn="urn:adsk.eagle:library:325" package="1X02" package3d_urn="urn:adsk.eagle:package:22435/2" value="" x="21.59" y="10.16" smashed="yes">
-<attribute name="NAME" x="18.9738" y="11.9888" size="1.27" layer="25" ratio="10"/>
-<attribute name="VALUE" x="19.05" y="6.985" size="1.27" layer="27"/>
-</element>
 <element name="QG1" library="crystal" library_urn="urn:adsk.eagle:library:204" package="DIL14S" package3d_urn="urn:adsk.eagle:package:12068/1" value="" x="54.61" y="17.78" smashed="yes" rot="R180">
 <attribute name="MF" value="" x="54.61" y="17.78" size="1.778" layer="27" rot="R180" display="off"/>
@@
 <contactref element="CPU" pad="2"/>
 <contactref element="RDY" pad="2"/>
-<contactref element="ROM-RDY" pad="1"/>
 <wire x1="30.48" y1="21.59" x2="29.21" y2="21.59" width="0.3048" layer="16"/>
 <wire x1="17.78" y1="33.02" x2="29.21" y2="21.59" width="0.3048" layer="16"/>
-<wire x1="20.32" y1="10.16" x2="19.05" y2="8.89" width="0.3048" layer="16"/>
 <wire x1="30.48" y1="21.59" x2="25.4" y2="21.59" width="0.3048" layer="1"/>
 <wire x1="25.4" y1="21.59" x2="21.59" y2="17.78" width="0.3048" layer="1"/>
 <via x="21.59" y="17.78" extent="1-16" drill="0.4"/>
-<wire x1="21.59" y1="17.78" x2="20.32" y2="16.51" width="0.3048" layer="16"/>
-<wire x1="20.32" y1="16.51" x2="20.32" y2="10.16" width="0.3048" layer="16"/>
 <wire x1="8.89" y1="35.56" x2="16.51" y2="35.56" width="0.3048" layer="16"/>
 <wire x1="16.51" y1="35.56" x2="17.78" y2="34.29" width="0.3048" layer="16"/>
 <wire x1="17.78" y1="34.29" x2="17.78" y2="33.02" width="0.3048" layer="16"/>
 <contactref element="SIG" pad="1"/>
-<wire x1="19.05" y1="8.89" x2="19.05" y2="3.175" width="0.3048" layer="16"/>
+<wire x1="21.59" y1="17.78" x2="19.05" y2="15.24" width="0.3048" layer="16"/>
+<wire x1="19.05" y1="15.24" x2="19.05" y2="3.175" width="0.3048" layer="16"/>
 </signal>
 <signal name="N$3">
@@
 <wire x1="5.21" y1="38.1" x2="5.08" y2="38.23" width="0.3048" layer="1"/>
 </signal>
-<signal name="N$8">
-<contactref element="EEPROM" pad="1"/>
-<contactref element="ROM-RDY" pad="2"/>
-<wire x1="81.28" y1="60.96" x2="78.74" y2="60.96" width="0.3048" layer="16"/>
-<wire x1="78.74" y1="60.96" x2="77.47" y2="59.69" width="0.3048" layer="16"/>
-<wire x1="77.47" y1="22.86" x2="74.93" y2="20.32" width="0.3048" layer="16"/>
-<via x="74.93" y="20.32" extent="1-16" drill="0.4"/>
-<wire x1="74.93" y1="20.32" x2="71.12" y2="16.51" width="0.3048" layer="1"/>
-<wire x1="77.47" y1="59.69" x2="77.47" y2="22.86" width="0.3048" layer="16"/>
-<wire x1="71.12" y1="16.51" x2="41.91" y2="16.51" width="0.3048" layer="1"/>
-<wire x1="41.91" y1="16.51" x2="36.83" y2="11.43" width="0.3048" layer="1"/>
-<wire x1="36.83" y1="11.43" x2="24.13" y2="11.43" width="0.3048" layer="1"/>
-<wire x1="24.13" y1="11.43" x2="22.86" y2="10.16" width="0.3048" layer="1"/>
-</signal>
 <signal name="N$9">
